Commit message: works fast now

File: URDF/mobileManipulator.urdf (robot description, URDF)
Before this commit: robot simplerobot_renamed, 7 links, 6 joints
Joints:
- joint joint_base_to_upper_arm: limit lower=-1.8 upper=1.8 effort=1000 velocity=0.5 -> lower=-1.8 upper=1.8 effort=1000 velocity=3
- joint joint_mobile_theta: limit effort=87 velocity=2 -> effort=1000 velocity=10
- joint joint_mobile_x: limit effort=87 velocity=2 -> effort=1000 velocity=10
- joint joint_mobile_y: limit effort=87 velocity=2 -> effort=1000 velocity=10
- joint joint_upper_to_lower_arm: limit lower=-2.1 upper=2.1 effort=1000 velocity=0.5 -> lower=-2.1 upper=2.1 effort=1000 velocity=3
